File: hardware/V2.0/humidity.kicad_pcb (KiCad board)
At the start: 2 copper layers, 15 x 25 mm, 24 parts, among them P101 CON-SENSOR2, P102 BOOT, P103 DEBUG, U101 XMC1XXX24, U102 SHT3x-DIS, U103 DRILL, U104 DRILL, U105 DRILL, U106 DRILL

Commit message: add description
Other:
- board text added: "Copyright Tinkerforge GmbH 2017. This documentation describes Open Hardware and is licensed under the CERN OHL v. 1.1. You may redistribute and modify this documentation under the terms of the CERN OHL v.1.1. (http://ohwr.org/cernohl). This documentation is distributed WITHOUT ANY EXPRESS OR IMPLIED WARRANTY, INCLUDING OF MERCHANTABILITY, SATISFACTORY QUALITY AND FITNESS FOR A PARTICULAR PURPOSE.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"
Changed lines of the file:
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@@
     (area 139.244999 127.644999 155.955001 154.355001)
     (thickness 1.6)
-    (drawings 12)
+    (drawings 13)
     (tracks 186)
     (zones 0)
@@
   )
   (page A4)
+  (title_block
+    (title "Humidity bricklet")
+    (date 2017-05-08)
+    (rev 2.0)
+    (company "Tinkerforge GmbH")
+    (comment 1 "Licensed under CERN OHL v.1.1")
+    (comment 2 "Copyright (©) 2017, B.Nordmeyer <bastian@tinkerforge.com>")
+  )
   (layers
     (0 F.Cu signal)
@@
       (net 17 "Net-(P103-Pad1)"))
   )
+  (gr_text "Copyright Tinkerforge GmbH 2017.\nThis documentation describes Open Hardware and is licensed under the\nCERN OHL v. 1.1.\nYou may redistribute and modify this documentation under the terms of the\nCERN OHL v.1.1. (http://ohwr.org/cernohl). This documentation is distributed\nWITHOUT ANY EXPRESS OR IMPLIED WARRANTY, INCLUDING OF\nMERCHANTABILITY, SATISFACTORY QUALITY AND FITNESS FOR A\nPARTICULAR PURPOSE. Please see the CERN OHL v.1.1 for applicable\nconditions" (at 257.15 155.8) (layer Cmts.User)
+    (effects (font (size 0.8 0.8) (thickness 0.2)))
+  )
   (gr_text 2.0 (at 150.1 134.9 90) (layer F.SilkS)
